Commit message: Use stl to have colors and fixed wheels position

File: hase_description/urdf/hase.urdf.xacro (robot description, xacro)
@@ -4,6 +4,6 @@
   <xacro:property name="wheelbase" value="0.0" />
   <xacro:property name="track" value="0.23" />
-  <xacro:property name="wheel_vertical_offset" value="0.0363" />
-  <xacro:property name="footprint_vertical_offset" value="0.0548" />
+  <xacro:property name="wheel_vertical_offset" value="0.0315" />
+  <xacro:property name="footprint_vertical_offset" value="0.05" />
   <xacro:property name="wheel_radius" value="0.0615" />
   <xacro:property name="wheel_width" value="0.0205" />
@@ -13,4 +13,6 @@
   <material name="dark_grey"><color rgba="0.2 0.2 0.2 1.0" /></material>
   <material name="light_grey"><color rgba="0.4 0.4 0.4 1.0" /></material>
+  <material name="light_green"><color rgba="0.0 0.4 0.0 1.0" /></material>
+  <material name="green"><color rgba="0.0 0.8 0.0 1.0" /></material>
   <material name="yellow"><color rgba="0.8 0.8 0.0 1.0" /></material>
   <material name="black"><color rgba="0.15 0.15 0.15 1.0" /></material>
@@ -21,7 +23,7 @@
         <origin xyz="0 0 0" rpy="0 0 0"/>
         <geometry>
-          <mesh filename="package://hase_description/meshes/wheel.dae" scale=".001 .001 .001"/>
+          <mesh filename="package://hase_description/meshes/wheel.stl" scale=".001 .001 .001"/>
         </geometry>
-        <material name="black" />
+        <material name="light_green" />
       </visual>
       <collision>
@@ -67,10 +69,10 @@
       <origin xyz="0 0 ${footprint_vertical_offset}" rpy="0 0 0"/>
       <geometry>
-        <mesh filename="package://hase_description/meshes/base.dae" scale=".001 .001 .001"/>
+        <mesh filename="package://hase_description/meshes/base.stl" scale=".001 .001 .001"/>
       </geometry>
-      <material name="yellow" />
+      <material name="black" />
     </visual>
     <collision>
-      <origin xyz="0.0 0 ${chassis_height/2}" rpy="0 0 0"/> <!-- should we use footprint_vertical?-->
+      <origin xyz="0.0 0 ${chassis_height/2}" rpy="0 0 0"/>
       <geometry>
         <cylinder length="${chassis_height}" radius="${chassis_radius}"/>

Commit message: Fix wheel transmission and orientation

File: hase_description/urdf/hase.urdf.xacro (robot description, xacro)
@@ -49,7 +49,15 @@
       <child link="${prefix}_wheel_link" />
       <xacro:insert_block name="joint_pose" />
-      <hardwareInterface>VelocityJointInterface</hardwareInterface>
       <axis xyz="0 0 1"/>
     </joint>
+    <transmission name="${prefix}_wheel_trans">
+      <type>transmission_interface/SimpleTransmission</type>
+      <joint name="${prefix}_wheel">
+        <hardwareInterface>VelocityJointInterface</hardwareInterface>
+      </joint>
+      <actuator name="${prefix}_actuator">
+        <mechanicalReduction>1</mechanicalReduction>
+      </actuator>
+    </transmission>
   </xacro:macro>
   <xacro:wheel prefix="left">
@@ -57,5 +65,5 @@
   </xacro:wheel>
   <xacro:wheel prefix="right">
-    <origin xyz="${wheelbase/2} ${-track/2} ${wheel_vertical_offset}" rpy="${PI/2} 0 0" />
+    <origin xyz="${wheelbase/2} ${-track/2} ${wheel_vertical_offset}" rpy="${-PI/2} 0 0" />
   </xacro:wheel>
   <link name="base_link"></link>

Commit message: Fix casters

File: hase_description/urdf/hase.urdf.xacro (robot description, xacro)
@@ -98,4 +98,11 @@
   </link>
   <link name="caster_front_link">
+    <visual>
+      <origin rpy="0 0 0" xyz="0 0 0"/>
+      <geometry>
+        <cylinder length="0.015" radius="0.04"/>
+      </geometry>
+      <material name="light_grey" />
+    </visual>
     <collision>
       <geometry>
@@ -115,12 +122,19 @@
     <parent link="chassis_link"/>
     <child link="caster_front_link"/>
-    <origin xyz="0.115 0.0 0.015" rpy="${-PI/2} 0 0"/>
+    <origin xyz="0.115 0.0 0.01" rpy="${-PI/2} 0 0"/>
   </joint>
   <joint name="caster_back_joint" type="fixed">
     <parent link="chassis_link"/>
     <child link="caster_back_link"/>
-    <origin xyz="-0.115 0.0 0.015" rpy="${-PI/2} 0 0"/>
+    <origin xyz="-0.115 0.0 0.01" rpy="${-PI/2} 0 0"/>
   </joint>
   <link name="caster_back_link">
+    <visual>
+      <origin rpy="0 0 0" xyz="0 0 0"/>
+      <geometry>
+        <cylinder length="0.015" radius="0.04"/>
+      </geometry>
+      <material name="light_grey" />
+    </visual>
     <collision>
       <geometry>

Commit message: hase_description: Initial attempt to add sick tim551

File: hase_description/urdf/hase.urdf.xacro (robot description, xacro)
@@ -90,9 +90,15 @@
       <!-- Center of mass -->
       <origin xyz="0 0 0"/>
-      <mass value="2.4"/> <!-- 2.4/2.6 kg for small/big battery pack -->
-      <!-- Moments of inertia: ( chassis without wheels ) -->
-      <inertia ixx="0.019995" ixy="0.0" ixz="0.0"
-               iyy="0.019995" iyz="0.0"
-               izz="0.03675" />
+      <mass value="2.4"/> <!--TODO: Set correct weight-->
+      <!-- Hase's inertia tensor is approximated by a cylinder with homogeneous mass distribution
+              More details: http://en.wikipedia.org/wiki/List_of_moment_of_inertia_tensors
+              m = 2.4 kg; h = 0.1 m; r = 0.175 m
+              ixx = 1/12 * m * (3 * r^2 + h^2)
+              iyy = 1/12 * m * (3 * r^2 + h^2)
+              izz = 1/2 * m * r^2
+      -->
+     <inertia ixx="0.020375" ixy="0.0" ixz="0.0"
+              iyy="0.020375" iyz="0.0"
+              izz="0.03675" />
     </inertial>
   </link>
@@ -153,3 +159,10 @@
   <!-- Bring in simulation data for Gazebo. -->
   <xacro:include filename="hase.gazebo" />
+  <joint name="laser_mount_link_joint" type="fixed">
+    <origin xyz="0 0 0.10" rpy="0 0 0" />
+    <parent link="base_link"/>
+    <child link="laser_mount_link" />
+  </joint>
+  <xacro:include filename="$(find sick_tim)/urdf/sick_tim.urdf.xacro" />
+  <xacro:sick_tim551 name="laser" ros_topic="front/scan" />
 </robot>

Commit message: hase_description: use simple base, add realistic ballcasters and move lidar

File: hase_description/urdf/hase.urdf.xacro (robot description, xacro)
@@ -5,8 +5,8 @@
   <xacro:property name="track" value="0.23" />
   <xacro:property name="wheel_vertical_offset" value="0.0315" />
-  <xacro:property name="footprint_vertical_offset" value="0.05" />
+  <xacro:property name="footprint_vertical_offset" value="0.003" />
   <xacro:property name="wheel_radius" value="0.0615" />
   <xacro:property name="wheel_width" value="0.0205" />
-  <xacro:property name="chassis_height" value="0.1" />
+  <xacro:property name="chassis_height" value="0.05" />
   <xacro:property name="chassis_radius" value="0.178" />
   <xacro:property name="dummy_inertia" value="1e-09"/>
@@ -18,4 +18,5 @@
   <material name="black"><color rgba="0.15 0.15 0.15 1.0" /></material>
   <material name="white"><color rgba="0.85 0.85 0.85 1.0" /></material>
+  <material name="acrilic"><color rgba="0.85 0.85 0.85 0.3" /></material>
   <xacro:macro name="wheel" params="prefix *joint_pose">
     <link name="${prefix}_wheel_link">
@@ -69,4 +70,41 @@
     <origin xyz="${wheelbase/2} ${-track/2} ${wheel_vertical_offset}" rpy="${-PI/2} 0 0" />
   </xacro:wheel>
+  <xacro:macro name="caster" params="prefix *joint_pose">
+    <link name="${prefix}_caster_link">
+      <visual>
+        <origin rpy="${PI} 0 ${PI/2}" xyz="0 0 -0.01125"/>
+        <geometry>
+          <mesh filename="package://hase_description/meshes/ball_caster.stl" scale=".001 .001 .001"/>
+        </geometry>
+        <material name="light_grey" />
+      </visual>
+      <collision>
+        <geometry>
+          <sphere radius="0.0075"/>
+        </geometry>
+        <origin rpy="0 0 0" xyz="0 0 -0.0225"/>
+      </collision>
+      <inertial>
+        <mass value="0.01" />
+        <origin xyz="0 0 0" />
+        <inertia ixx="0.001" ixy="0.0" ixz="0.0"
+                 iyy="0.001" iyz="0.0"
+                 izz="0.001" />
+      </inertial>
+    </link>
+    <joint name="${prefix}_caster_joint" type="fixed">
+      <parent link="chassis_link"/>
+      <child link="${prefix}_caster_link"/>
+      <xacro:insert_block name="joint_pose" />
+      <axis xyz="0 0 1"/>
+      <!--origin xyz="0.16 0.0 0" rpy="0 0 0"/-->
+    </joint>
+  </xacro:macro>
+  <xacro:caster prefix="front">
+    <origin xyz="0.155 0 0" rpy="0 0 0" />
+  </xacro:caster>
+  <xacro:caster prefix="back">
+    <origin xyz="-0.155 0 0" rpy="0 0 0" />
+  </xacro:caster>
   <link name="base_link"></link>
   <joint name="base_link_joint" type="fixed">
@@ -79,7 +117,7 @@
       <origin xyz="0 0 ${footprint_vertical_offset}" rpy="0 0 0"/>
       <geometry>
-        <mesh filename="package://hase_description/meshes/base.stl" scale=".001 .001 .001"/>
+        <mesh filename="package://hase_description/meshes/base_simple.stl" scale=".001 .001 .001"/>
       </geometry>
-      <material name="black" />
+      <material name="acrilic" />
     </visual>
     <collision>
@@ -105,62 +143,8 @@
     </inertial>
   </link>
-  <link name="caster_front_link">
-    <visual>
-      <origin rpy="0 0 0" xyz="0 0 0"/>
-      <geometry>
-        <cylinder length="0.015" radius="0.04"/>
-      </geometry>
-      <material name="light_grey" />
-    </visual>
-    <collision>
-      <geometry>
-        <cylinder length="0.015" radius="0.04"/>
-      </geometry>
-      <origin rpy="0 0 0" xyz="0 0 0"/>
-    </collision>
-    <inertial>
-      <mass value="0.01" />
-      <origin xyz="0 0 0" />
-      <inertia ixx="0.001" ixy="0.0" ixz="0.0"
-               iyy="0.001" iyz="0.0"
-               izz="0.001" />
-    </inertial>
-  </link>
-  <joint name="caster_front_joint" type="fixed">
-    <parent link="chassis_link"/>
-    <child link="caster_front_link"/>
-    <origin xyz="0.115 0.0 0.01" rpy="${-PI/2} 0 0"/>
-  </joint>
-  <joint name="caster_back_joint" type="fixed">
-    <parent link="chassis_link"/>
-    <child link="caster_back_link"/>
-    <origin xyz="-0.115 0.0 0.01" rpy="${-PI/2} 0 0"/>
-  </joint>
-  <link name="caster_back_link">
-    <visual>
-      <origin rpy="0 0 0" xyz="0 0 0"/>
-      <geometry>
-        <cylinder length="0.015" radius="0.04"/>
-      </geometry>
-      <material name="light_grey" />
-    </visual>
-    <collision>
-      <geometry>
-        <cylinder length="0.015" radius="0.04"/>
-      </geometry>
-      <origin rpy="0 0 0" xyz="0 0 0"/>
-    </collision>
-    <inertial>
-      <mass value="0.01" />
-      <origin xyz="0 0 0" />
-      <inertia ixx="0.001" ixy="0.0" ixz="0.0"
-               iyy="0.001" iyz="0.0"
-               izz="0.001" />
-    </inertial>
-  </link>
   <!-- Bring in simulation data for Gazebo. -->
   <xacro:include filename="hase.gazebo" />
   <joint name="laser_mount_link_joint" type="fixed">
-    <origin xyz="0 0 0.10" rpy="0 0 0" />
+    <origin xyz="0.135 0 0.006" rpy="0 0 0" />
     <parent link="base_link"/>
     <child link="laser_mount_link" />

Commit message: hase_description: add motor and bracket

File: hase_description/urdf/hase.urdf.xacro (robot description, xacro)
@@ -143,4 +143,27 @@
     </inertial>
   </link>
+  <xacro:macro name="motor" params="prefix *joint_pose">
+    <link name="${prefix}_motor_link">
+      <visual>
+        <origin rpy="${PI/2} 0 0" xyz="0 0 0.026"/>
+        <geometry>
+          <mesh filename="package://hase_description/meshes/motor_and_bracket.stl" scale=".001 .001 .001"/>
+        </geometry>
+        <material name="light_grey" />
+      </visual>
+    </link>
+    <joint name="${prefix}_motor_joint" type="fixed">
+      <parent link="chassis_link"/>
+      <child link="${prefix}_motor_link"/>
+      <xacro:insert_block name="joint_pose" />
+      <axis xyz="0 0 1"/>
+    </joint>
+  </xacro:macro>
+  <xacro:motor prefix="left">
+    <origin xyz="0 -0.05 0" rpy="0 0 0" />
+  </xacro:motor>
+  <xacro:motor prefix="right">
+    <origin xyz="0 0.05 0" rpy="0 0 ${PI}" />
+  </xacro:motor>
   <!-- Bring in simulation data for Gazebo. -->
   <xacro:include filename="hase.gazebo" />
